File: circuitPanneauCarbOnFire/circuitPanneauCarbOnFire.sch (KiCad schematic (older format))
At the start: 13 parts, among them SW1 SW_DIP_x01, SW2 SW_DIP_x01

Commit message: circuit electrique grove+capteur+panneauAvant
Parts:
- removed D1, D2: LED, LED_THT:LED_D5.0mm_IRGrey, symbol Device:LED
- removed SW1, SW2: SW_DIP_x01, Button_Switch_THT:SW_DIP_SPSTx01_Slide_9.78x4.72mm_W7.62mm_P2.54mm, symbol Switch:SW_DIP_x01
- removed UFusible1, Ualphasense1: molex2pin, Connector_Molex:Molex_KK-254_AE-6410-02A_1x02_P2.54mm_Vertical, symbol LibrairieCarbonEye:molex2pin
- removed UIn1, Uout1: connecteurCC12V, Button_Switch_THT:SW_DIP_SPSTx01_Slide_9.78x4.72mm_W7.62mm_P2.54mm, symbol LibrairieCarbonEye:connecteurCC12V
- added J1: Screw_Terminal_01x14, TerminalBlock_Phoenix:TerminalBlock_Phoenix_MKDS-1,5-14-5.08_1x14_P5.08mm_Horizontal, symbol Connector:Screw_Terminal_01x14
- added J2, J3: 4P4C, Connector:NS-Tech_Grove_1x04_P2mm_Vertical, symbol Connector:4P4C
- added J4: Conn_01x10_Male, Connector_Molex:Molex_Micro-Latch_53253-1070_1x10_P2.00mm_Vertical, symbol Connector:Conn_01x10_Male
- added J5: Conn_01x02_Male, Connector_Molex:Molex_KK-254_AE-6410-02A_1x02_P2.54mm_Vertical, symbol Connector:Conn_01x02_Male
- added J6: 4P4C, Connector_Molex:Molex_SL_171971-0004_1x04_P2.54mm_Vertical, symbol Connector:4P4C
- added R3: 220, Resistor_THT:R_Axial_DIN0207_L6.3mm_D2.5mm_P10.16mm_Horizontal, symbol Device:R
- added R4: 100, Resistor_THT:R_Axial_DIN0207_L6.3mm_D2.5mm_P10.16mm_Horizontal, symbol Device:R
- UalimArduino1: renamed from Uarduino1; symbol LibrairieCarbonEye:molex2pin -> circuitPanneauCarbOnFire-rescue:molex2pin-LibrairieCarbonEye
Connections:
- net Fusible1: now reaches R1.1, UalimArduino1.1
- net Fusible1: now also J1.1 (Pin_1), J5.1 (Pin_1), J6.4
- net SwitchOut2: now reaches C1.1, DRoueLibre1.2 (A), R2.1
- net SwitchOut2: now also J1.6 (Pin_6), J1.7 (Pin_7)
- net GND: now reaches C1.2, DRoueLibre1.1 (K)
- net GND: now also UalimArduino1.2, J1.11 (Pin_11), J1.12 (Pin_12), J1.13 (Pin_13), J1.14 (Pin_14), J2.1, J3.1, J4.2 (Pin_2), J6.3, R4.2
- net CatLedOut: now reaches R2.2
- net CatLedOut: now also J1.3 (Pin_3)
- net CatLedIn: now reaches R1.2
- net CatLedIn: now also J1.2 (Pin_2)
- new net: J6.2, R3.2
- new net A0: J4.7 (Pin_7), J5.2 (Pin_2), R4.1
- new net A1: J4.8 (Pin_8), J6.1, R3.1
- new net Fusible2: J1.4 (Pin_4), J1.5 (Pin_5)
- new net SCL: J2.4, J3.4, J4.3 (Pin_3)
- new net SDA: J2.3, J3.3, J4.4 (Pin_4)
- new net SwitchIn1: J1.10 (Pin_10), J1.8 (Pin_8), J1.9 (Pin_9)
- new net Vdd: J2.2, J3.2, J4.1 (Pin_1)
- no-connect marks 0 -> 4
