File: PCB/circuitPanneauCarbOnFire.kicad_pcb (KiCad board)
At the start: 2 copper layers, 73.7 x 38.1 mm, 15 parts, among them J1 Screw_Terminal_01x14, J2 4P4C, J3 4P4C, J4 Conn_01x10_Male, J5 Conn_01x02_Male, J6 4P4C

Commit message: pcb + script python
Parts:
- J1: footprint TerminalBlock_Phoenix:TerminalBlock_Phoenix_MKDS-1,5-14-5.08_1x14_P5.08mm_Horizontal -> TerminalBlock_Phoenix:TerminalBlock_Phoenix_PT-1,5-14-5.0-H_1x14_P5.00mm_Horizontal
- J4: footprint Connector_Molex:Molex_Micro-Latch_53253-1070_1x10_P2.00mm_Vertical -> Connector_PinSocket_2.54mm:PinSocket_1x10_P2.54mm_Vertical
- moved J4 4.40 mm to (152.8, 67.3), turned to 270 degrees
- moved J1 0.87 mm to (98.5, 75.3)
Routing:
- net AnoLedIn: track 192.6 -> 7.53 mm
- net SwitchOut2: track 115.3 -> 108.6 mm
- net A1: track 17.1 -> 20.5 mm
- net Vdd: track 29.0 -> 26.4 mm
- net SDA: track 55.4 -> 57.1 mm
- net Fusible1: track 46.6 -> 48.0 mm
- net A0: track 33.9 -> 35.0 mm
- net CatLedIn: track 9.20 -> 9.97 mm
- added copper zone on B.Cu, net AnoLedIn
- removed copper zone on F.Cu, net AnoLedIn
Other:
- net class Default: clearance 0.4 -> 0.6
- rule trace_clearance: 0.4 -> 0.6
- board text added: "CarbOnFire"
